File: pv_monitor.kicad_sch (KiCad schematic)
At the start: 76 parts, among them J1 Raspberry_Pi_2_3, J10 cell in current, J11 cell out current, J2 balancer alarm, J3 spare, J4 heating, J5 trip_rcd, J9 battery, K1 RT424024, K2 RT424024, Q1 DMG3402L, Q2 DMG3402L, U2 LM73

Commit message: 1st revision ready to order
Parts:
- removed J2: balancer alarm, TerminalBlock_WAGO:TerminalBlock_WAGO_236-102_1x02_P5.00mm_45Degree, symbol Connector:Screw_Terminal_01x02
- removed TP1, TP2: ~, symbol Connector:TestPoint
- added J6: balancer, TerminalBlock_WAGO:TerminalBlock_WAGO_236-103_1x03_P5.00mm_45Degree, symbol Connector:Screw_Terminal_01x03
- added TP10, TP11, TP7, TP8, TP9: TestPoint, TestPoint:TestPoint_THTPad_D2.0mm_Drill1.0mm, symbol Connector:TestPoint
- C1: renamed from C12; footprint (none) -> Capacitor_SMD:C_0805_2012Metric_Pad1.18x1.45mm_HandSolder
- C10: renamed from C2; footprint (none) -> Capacitor_SMD:C_0805_2012Metric_Pad1.18x1.45mm_HandSolder
- C11: renamed from C4; footprint (none) -> Capacitor_SMD:C_Elec_8x10.2; ManufacturerPartNumber (none) -> EEH-ZK1V101XV
- C12: renamed from C6; footprint (none) -> Capacitor_SMD:C_0805_2012Metric_Pad1.18x1.45mm_HandSolder
- C2: renamed from C11; footprint (none) -> Capacitor_SMD:C_0805_2012Metric_Pad1.18x1.45mm_HandSolder
- C3: renamed from C8; footprint (none) -> Capacitor_SMD:C_1206_3216Metric_Pad1.33x1.80mm_HandSolder
- C4: renamed from C9; footprint (none) -> Capacitor_SMD:C_1206_3216Metric_Pad1.33x1.80mm_HandSolder
- C5: renamed from C10; footprint (none) -> Capacitor_SMD:C_1206_3216Metric_Pad1.33x1.80mm_HandSolder
- C6: renamed from C7; footprint (none) -> Capacitor_SMD:C_0805_2012Metric_Pad1.18x1.45mm_HandSolder
- C7: renamed from C3; footprint (none) -> Capacitor_SMD:C_Elec_8x10.2; ManufacturerPartNumber (none) -> EEH-ZK1V101XV
- C8: renamed from C5; footprint (none) -> Capacitor_SMD:C_0805_2012Metric_Pad1.18x1.45mm_HandSolder
- C9: renamed from C1; footprint (none) -> Capacitor_SMD:C_0805_2012Metric_Pad1.18x1.45mm_HandSolder
- D3, D4: footprint (none) -> Diode_SMD:D_SMA_Handsoldering
- J7: renamed from J1; footprint (none) -> Module:Raspberry_Pi_Zero_Socketed_THT_FaceDown_MountingHoles
- JP1: footprint (none) -> Connector_PinSocket_2.54mm:PinSocket_1x02_P2.54mm_Vertical
- R1: renamed from R9; value R -> 150k; footprint (none) -> Resistor_SMD:R_0805_2012Metric_Pad1.20x1.40mm_HandSolder
- R10: renamed from R17; footprint (none) -> Resistor_SMD:R_0805_2012Metric_Pad1.20x1.40mm_HandSolder
- R11: renamed from R18; footprint (none) -> Resistor_SMD:R_0805_2012Metric_Pad1.20x1.40mm_HandSolder
- R12: renamed from R7; footprint (none) -> Resistor_SMD:R_0805_2012Metric_Pad1.20x1.40mm_HandSolder
- R13: renamed from R3; footprint (none) -> Resistor_SMD:R_0805_2012Metric_Pad1.20x1.40mm_HandSolder
- R14: renamed from R1; value R -> 10k; footprint (none) -> Resistor_SMD:R_0805_2012Metric_Pad1.20x1.40mm_HandSolder
- R15: renamed from R19; footprint (none) -> Resistor_SMD:R_0805_2012Metric_Pad1.20x1.40mm_HandSolder
- R16: renamed from R20; footprint (none) -> Resistor_SMD:R_0805_2012Metric_Pad1.20x1.40mm_HandSolder
- R17: renamed from R5; footprint (none) -> Resistor_SMD:R_0805_2012Metric_Pad1.20x1.40mm_HandSolder
- R18: renamed from R4; footprint (none) -> Resistor_SMD:R_0805_2012Metric_Pad1.20x1.40mm_HandSolder
- R19: renamed from R2; footprint (none) -> Resistor_SMD:R_0805_2012Metric_Pad1.20x1.40mm_HandSolder
- R2: renamed from R12; value R -> 100k; footprint (none) -> Resistor_SMD:R_0805_2012Metric_Pad1.20x1.40mm_HandSolder
- R20: renamed from R6; footprint (none) -> Resistor_SMD:R_0805_2012Metric_Pad1.20x1.40mm_HandSolder
- R3: renamed from R10; value R -> 150k; footprint (none) -> Resistor_SMD:R_0805_2012Metric_Pad1.20x1.40mm_HandSolder
- R4: renamed from R13; value R -> 100k; footprint (none) -> Resistor_SMD:R_0805_2012Metric_Pad1.20x1.40mm_HandSolder
- R5: renamed from R8; footprint (none) -> Resistor_SMD:R_0805_2012Metric_Pad1.20x1.40mm_HandSolder
- R6: renamed from R11; value R -> 120k; footprint (none) -> Resistor_SMD:R_0805_2012Metric_Pad1.20x1.40mm_HandSolder
- R7: renamed from R14; value R -> 20k; footprint (none) -> Resistor_SMD:R_0805_2012Metric_Pad1.20x1.40mm_HandSolder
- R8: renamed from R15; value R -> 130k; footprint (none) -> Resistor_SMD:R_0805_2012Metric_Pad1.20x1.40mm_HandSolder
- R9: renamed from R16; value R -> 10k; footprint (none) -> Resistor_SMD:R_0805_2012Metric_Pad1.20x1.40mm_HandSolder
- RV1: footprint (none) -> Potentiometer_THT:Potentiometer_Piher_PT-10-V10_Vertical
- TP1: renamed from TP12; footprint (none) -> TestPoint:TestPoint_THTPad_D2.0mm_Drill1.0mm
- TP12: renamed from TP3; footprint (none) -> TestPoint:TestPoint_THTPad_D2.0mm_Drill1.0mm
- TP13: renamed from TP4; footprint (none) -> TestPoint:TestPoint_THTPad_D2.0mm_Drill1.0mm
- TP14: renamed from TP5; footprint (none) -> TestPoint:TestPoint_THTPad_D2.0mm_Drill1.0mm
- TP15: renamed from TP6; footprint (none) -> TestPoint:TestPoint_THTPad_D2.0mm_Drill1.0mm
- TP16: renamed from TP7; footprint (none) -> TestPoint:TestPoint_THTPad_D2.0mm_Drill1.0mm
- TP17: renamed from TP8; footprint (none) -> TestPoint:TestPoint_THTPad_D2.0mm_Drill1.0mm
- TP18: renamed from TP9; footprint (none) -> TestPoint:TestPoint_THTPad_D2.0mm_Drill1.0mm
- TP19: renamed from TP10; footprint (none) -> TestPoint:TestPoint_THTPad_D2.0mm_Drill1.0mm
- TP2: renamed from TP13; footprint (none) -> TestPoint:TestPoint_THTPad_D2.0mm_Drill1.0mm
- TP3: renamed from TP11; footprint (none) -> TestPoint:TestPoint_THTPad_D2.0mm_Drill1.0mm
- TP4: renamed from TP14; footprint (none) -> TestPoint:TestPoint_THTPad_D2.0mm_Drill1.0mm
- TP5: renamed from TP15; footprint (none) -> TestPoint:TestPoint_THTPad_D2.0mm_Drill1.0mm
- TP6: renamed from TP16; footprint (none) -> TestPoint:TestPoint_THTPad_D2.0mm_Drill1.0mm
- renumbered BT3 to BT1, BT1 to BT2, BT4 to BT3, BT2 to BT4, J11 to J1, J10 to J2, J9 to J3, J3 to J4, J4 to J5, J5 to J8, U3 to U1, U4 to U2, U2 to U3, U1 to U4
Connections:
- net GND: now also RV1.1, J6.3 (Pin_3); no longer RV1.3
- net balancer_alarm: now also J7.13 (GPIO27), J6.2 (Pin_2); no longer J7.15 (GPIO22)
- net cs_b: now also TP9.1
- net heating: now also J7.11 (GPIO17); no longer J7.37 (GPIO26)
- net i_cell_in: now also U2.7 (S4); no longer U2.4 (S1)
- net i_cell_out: now also U2.6 (S3); no longer U2.5 (S2)
- net miso: now also TP10.1
- net mux_addr_0: now also J7.40 (GPIO21/SCLK1); no longer J7.16 (GPIO23)
- net mux_addr_1: now also J7.38 (GPIO20/MOSI1); no longer J7.18 (GPIO24)
- net mux_addr_2: now also J7.35 (GPIO19/MISO1); no longer J7.22 (GPIO25)
- net scl: now also TP8.1
- net sclk: now also TP11.1
- net sda: now also TP7.1
- net trip_rcd: now also J7.12 (GPIO18/PWM0); no longer J7.13 (GPIO27)
- net v_cell_hi: now also U2.4 (S1); no longer U2.7 (S4)
- net v_cell_mid: now also U2.5 (S2); no longer U2.6 (S3)
- net at C9.2, R19.2, U4.6 (FB): now also RV1.3; no longer RV1.1
- no-connect marks 0 -> 29
Other:
- moved on the sheet: TP3
